File: KiCad/SolarPowerBank.kicad_sch (KiCad schematic)
At the start: 31 parts, among them J1 Solar, J2 JST PH2, J3 Conn_01x04, J4 USB_A, U1 SW2303, U2 BQ25185

Commit message: Changed footprints to allow for easier hand soldering
Parts:
- U1: footprint Package_DFN_QFN:QFN-16-1EP_4x4mm_P0.65mm_EP2.15x2.15mm_ThermalVias -> SolarPowerBankLibrary:QFN-16-1EP_4x4mm_P0.65mm_EP2.15x2.15mm_ThermalVias-HandSolder
- U2: footprint SolarPowerBankLibrary:WSON-10-1EP_2.2x2.0mm_P0.4_ThermalVias -> SolarPowerBankLibrary:WSON-10-1EP_2.2x2.0mm_P0.4_ThermalVias-HandSolder
Changed lines of the file:
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@@
 	(label "VBUS"
 		(at 257.81 44.45 90)
-		(fields_autoplaced yes)
 		(effects
 			(font
@@
 	(label "VDD"
 		(at 177.8 119.38 0)
-		(fields_autoplaced yes)
 		(effects
 			(font
@@
 	(label "SYS"
 		(at 143.51 54.61 0)
-		(fields_autoplaced yes)
 		(effects
 			(font
@@
 	(label "SYS"
 		(at 97.79 82.55 180)
-		(fields_autoplaced yes)
 		(effects
 			(font
@@
 	(label "IFB"
 		(at 210.82 116.84 0)
-		(fields_autoplaced yes)
 		(effects
 			(font
@@
 	(label "SYS"
 		(at 180.34 60.96 0)
-		(fields_autoplaced yes)
 		(effects
 			(font
@@
 	(label "SYS"
 		(at 44.45 130.81 90)
-		(fields_autoplaced yes)
 		(effects
 			(font
@@
 	(label "DP"
 		(at 177.8 121.92 0)
-		(fields_autoplaced yes)
 		(effects
 			(font
@@
 	(label "CHG"
 		(at 97.79 85.09 180)
-		(fields_autoplaced yes)
 		(effects
 			(font
@@
 	(label "SYS"
 		(at 93.98 44.45 0)
-		(fields_autoplaced yes)
 		(effects
 			(font
@@
 	(label "DM"
 		(at 191.77 134.62 90)
-		(fields_autoplaced yes)
 		(effects
 			(font
@@
 	(label "SYS"
 		(at 176.53 93.98 0)
-		(fields_autoplaced yes)
 		(effects
 			(font
@@
 	(label "VBUS"
 		(at 227.33 60.96 180)
-		(fields_autoplaced yes)
 		(effects
 			(font
@@
 	(label "DM"
 		(at 250.19 44.45 90)
-		(fields_autoplaced yes)
 		(effects
 			(font
@@
 	(label "GATE"
 		(at 177.8 116.84 0)
-		(fields_autoplaced yes)
 		(effects
 			(font
@@
 	(label "FB"
 		(at 196.85 100.33 270)
-		(fields_autoplaced yes)
 		(effects
 			(font
@@
 	(label "CHG"
 		(at 48.26 52.07 0)
-		(fields_autoplaced yes)
 		(effects
 			(font
@@
 	(label "VDD"
 		(at 196.85 134.62 90)
-		(fields_autoplaced yes)
 		(effects
 			(font
@@
 	(label "DP"
 		(at 252.73 44.45 90)
-		(fields_autoplaced yes)
 		(effects
 			(font
@@
 	(label "FAULT"
 		(at 97.79 87.63 180)
-		(fields_autoplaced yes)
 		(effects
 			(font
@@
 	(label "GATE"
 		(at 180.34 68.58 0)
-		(fields_autoplaced yes)
 		(effects
 			(font
@@
 	(label "VBUS"
 		(at 199.39 100.33 270)
-		(fields_autoplaced yes)
 		(effects
 			(font
@@
 	(label "FB"
 		(at 158.75 64.77 0)
-		(fields_autoplaced yes)
 		(effects
 			(font
@@
 	(label "FAULT"
 		(at 48.26 49.53 0)
-		(fields_autoplaced yes)
 		(effects
 			(font
@@
 			)
 		)
-		(property "Footprint" "SolarPowerBankLibrary:WSON-10-1EP_2.2x2.0mm_P0.4_ThermalVias"
+		(property "Footprint" "SolarPowerBankLibrary:WSON-10-1EP_2.2x2.0mm_P0.4_ThermalVias-HandSolder"
 			(at 84.328 31.242 0)
 			(effects
@@
 			)
 		)
-		(property "Footprint" "Package_DFN_QFN:QFN-16-1EP_4x4mm_P0.65mm_EP2.15x2.15mm_ThermalVias"
+		(property "Footprint" "SolarPowerBankLibrary:QFN-16-1EP_4x4mm_P0.65mm_EP2.15x2.15mm_ThermalVias-HandSolder"
 			(at 195.072 151.384 0)
 			(effects
